Commit message: added launch_robot.launch.py

File: urdf/ercole.urdf.xacro (robot description, xacro)
@@ -1,14 +1,6 @@
 <?xml version="1.0"?>
-<robot xmlns:xacro="http://www.ros.org/wiki/xacro" name="ercole">
-    <xacro:arg name="use_ros2_control" default="true"/>
-    <xacro:arg name="sim_mode" default="false"/>
+<robot name="ercole" xmlns:xacro="http://www.ros.org/wiki/xacro">
     <xacro:include filename="common_properties.xacro" />
     <xacro:include filename="mobile_base.xacro" />
-    <xacro:if value="$(arg use_ros2_control)">
-        <xacro:include filename="ercole.ros2_control.xacro" />
-    </xacro:if>
-    <xacro:unless value="$(arg use_ros2_control)">
-        <xacro:include filename="ercole.gazebo.xacro" />
-    </xacro:unless>
     <xacro:include filename="lidar.xacro" />
 </robot>

File: urdf/ercole_rover.urdf.xacro (robot description, xacro)
@@ -12,8 +12,8 @@
     <xacro:include filename="ercole.gazebo.xacro" />
     <!-- Import Ercole ros2_control description  -->
-    <xacro:include filename="ercole.ros2_control_.xacro" />
-    <xacro:ercole
+    <xacro:include filename="ercole.ros2_control.xacro" />
+    <!-- <xacro:ercole
         model="$(arg model)" prefix="$(arg prefix)">
-    </xacro:ercole>
+    </xacro:ercole>  -->
     <xacro:if value="$(arg use_gazebo)">
         <xacro:ercole_gazebo model="$(arg model)" prefix="$(arg prefix)" />

File: urdf/gazebo_control.xacro (robot description, xacro)
@@ -1,5 +1,4 @@
 <?xml version="1.0"?>
 <robot xmlns:xacro="http://www.ros.org/wiki/xacro">
-    <xacro:macro name="ercole_gazebo" params="model prefix">
         <gazebo reference="base_link">
             <material>Gazebo/Blue</material>
@@ -30,4 +29,3 @@
             </plugin>
         </gazebo>
-     </xacro:macro>
 </robot>

File: urdf/ros2_control.xacro (robot description, xacro)
@@ -3,14 +3,7 @@
     <xacro:unless value="$(arg sim_mode)">
         <ros2_control name="RealRobot" type="system">
-            <hardware>
-                <plugin>diffdrive_arduino/DiffDriveArduino</plugin>
-                <param name="left_wheel_name">base_rl_wheel_joint</param>
-                <param name="right_wheel_name">base_rr_wheel_joint</param>
-                <param name="loop_rate">30</param>
-                <param name="device">/dev/ttyUSB0</param>
-                <param name="baud_rate">57600</param>
-                <param name="timeout">1000</param>
-                <param name="enc_counts_per_rev">3436</param>
-            </hardware>
+            <!-- <hardware>
+                <plugin>fake_components/GenericSystem</plugin>
+            </hardware> -->
             <joint name="base_rl_wheel_joint">
                 <command_interface name="velocity">

File: urdf/ros2_control_.xacro (robot description, xacro)
@@ -4,5 +4,12 @@
         <ros2_control name="RealRobot" type="system">
             <hardware>
-                <plugin>fake_components/GenericSystem</plugin>
+                <plugin>diffdrive_arduino/DiffDriveArduino</plugin>
+                <param name="left_wheel_name">base_rl_wheel_joint</param>
+                <param name="right_wheel_name">base_rr_wheel_joint</param>
+                <param name="loop_rate">30</param>
+                <param name="device">/dev/ttyUSB0</param>
+                <param name="baud_rate">57600</param>
+                <param name="timeout">1000</param>
+                <param name="enc_counts_per_rev">3436</param>
             </hardware>
             <joint name="base_rl_wheel_joint">
